Commit message: update

File: ur5/rom_ur_sim/urdf/ur5_camera.urdf.xacro (robot description, xacro)
@@ -45,6 +45,6 @@
    <xacro:arg name="use_fake_hardware" default="false" />
    <xacro:arg name="fake_sensor_commands" default="false" />
-   <xacro:arg name="sim_gazebo" default="true" />
-   <xacro:arg name="sim_ignition" default="false" />
+   <xacro:arg name="sim_gazebo" default="false" />
+   <xacro:arg name="sim_ignition" default="true" />
    <xacro:arg name="simulation_controllers" default="$(find rom_ur_sim)/config/ur5_controllers.yaml" />
    <!-- initial position for simulations (Fake Hardware, Gazebo, Ignition) -->
@@ -118,5 +118,5 @@
      trajectory_port="$(arg trajectory_port)"
      >
-     <origin xyz="0 0 0.8" rpy="0 0 0" />          <!-- position robot in the world -->
+     <origin xyz="0 0 0" rpy="0 0 0" />          <!-- position robot in the world -->
    </xacro:ur_robot>
    <xacro:if value="$(arg sim_gazebo)">

File: ur5/rom_ur_sim/urdf/ur5_camera_gripper.urdf.xacro (robot description, xacro)
@@ -43,6 +43,6 @@
    <xacro:arg name="use_fake_hardware" default="false" />
    <xacro:arg name="fake_sensor_commands" default="false" />
-   <xacro:arg name="sim_gazebo" default="true" />
-   <xacro:arg name="sim_ignition" default="false" />
+   <xacro:arg name="sim_gazebo" default="false" />
+   <xacro:arg name="sim_ignition" default="true" />
    <xacro:arg name="simulation_controllers" default="$(find rom_ur_sim)/config/ur5_controllers_gripper.yaml" />
    <!-- initial position for simulations (Fake Hardware, Gazebo, Ignition) -->
@@ -116,5 +116,5 @@
      trajectory_port="$(arg trajectory_port)"
      >
-     <origin xyz="0 0 0.8" rpy="0 0 0" />          <!-- position robot in the world -->
+     <origin xyz="0 0 0" rpy="0 0 0" />          <!-- position robot in the world -->
    </xacro:ur_robot>
    <xacro:if value="$(arg sim_gazebo)">
