Commit message: add table rviz,moveit planning ok

File: ur5/rom_ur_sim/urdf/ur5_camera_gripper.urdf.xacro (robot description, xacro)
@@ -116,5 +116,5 @@
      trajectory_port="$(arg trajectory_port)"
      >
-     <origin xyz="0 0 0" rpy="0 0 0" />          <!-- position robot in the world -->
+     <origin xyz="0 0 1.02" rpy="0 0 0" />          <!-- position robot in the world -->
    </xacro:ur_robot>
    <xacro:if value="$(arg sim_gazebo)">

Commit message: gz camera update

File: ur5/rom_ur_sim/urdf/ur5_camera_gripper.urdf.xacro (robot description, xacro)
@@ -4,5 +4,5 @@
    <xacro:arg name="name" default="ur"/>
    <!-- import main macro -->
-   <xacro:include filename="$(find rom_ur_sim)/urdf/camera_ign.xacro"/>
+   <!-- <xacro:include filename="$(find rom_ur_sim)/urdf/camera_ign.xacro"/> -->
    <xacro:include filename="$(find rom_ur_sim)/urdf/ur5_macro.xacro"/>
    <xacro:include filename="$(find ur_simulation_gz)/urdf/ur_gz.ros2_control.xacro" />
@@ -60,5 +60,5 @@
     force_abs_paths="true"
     >
-    <origin xyz="0 0 0" rpy="0 0 0" />          <!-- position robot in the world -->
+    <origin xyz="0 0 1.02" rpy="0 0 0" />          <!-- position robot in the world -->
   </xacro:ur_robot>
   <gazebo reference="world">
