Commit message: unstable

File: ur5/rom_ur_sim/urdf/camera.xacro (robot description, xacro)
@@ -29,6 +29,10 @@
         <parent link="base_link"/>
         <child link="camera_link"/>
-        <origin xyz="0.5 0 1.2" rpy="0 1.57 0" />
+        <origin xyz="0.2 0.6 1.2" rpy="0 1.570796326 0" />
     </joint>
+    <!-- <xacro:camera_v0 parent="panda_link0">
+	    <origin xyz="0.2 0.6 0.7" rpy="0 ${PI/2} 0"/>
+    </xacro:camera_v0>
+    <xacro:camera_gazebo_v0/> -->
     <link name="camera_optical_link"></link>
     <joint name="camera_optical_joint" type="fixed">

File: ur5/rom_ur_sim/urdf/camera_ign.xacro (robot description, xacro)
@@ -29,5 +29,5 @@
         <parent link="base_link"/>
         <child link="camera_link"/>
-        <origin xyz="0.5 0 0.7" rpy="0 1.57 0" />
+        <origin xyz="0.2 0.6 1.2" rpy="0 1.570796326 0" />
     </joint>
     <link name="camera_optical_link"></link>
@@ -69,8 +69,8 @@
             <pose> 0 0 0 0 0 0 </pose>
             <visualize>true</visualize>
-            <update_rate>10</update_rate>
+            <update_rate>30.0</update_rate>
             <camera>
                 <camera_info_topic>camera/camera_info</camera_info_topic>
-                <horizontal_fov>1.089</horizontal_fov>
+                <horizontal_fov>1.8</horizontal_fov>
                 <image>
                     <format>R8G8B8</format>
@@ -79,7 +79,12 @@
                 </image>
                 <clip>
-                    <near>0.05</near>
-                    <far>8.0</far>
+                    <near>0.02</near>
+                    <far>300</far>
                 </clip>
+                <noise>
+                <type>gaussian</type>
+                <mean>0.0</mean>
+                <stddev>0.007</stddev>
+              </noise>
             </camera>
             <topic>camera/image_raw</topic>
