Commit message: camera ok, to do depth camera,fixed camera tf for yolo

File: ur5/rom_ur_sim/urdf/camera_ign.xacro (robot description, xacro)
@@ -1,5 +1,5 @@
 <?xml version="1.0"?>
 <robot xmlns:xacro="http://ros.org/wiki/xacro">
-    <material name="blue">
+    <material name="Blue">
         <color rgba="0 0 1 1"/>
     </material>
@@ -44,8 +44,7 @@
                 </mesh>
             </geometry>
-            <material>Gazebo/Red</material>
+            <material>Gazebo/Blue</material>
         </visual>
-        <!-- <material>Gazebo/Red</material> -->
-        <sensor name="camera" type="depth">
+        <!-- <sensor name="camera" type="depth">
             <pose> 0 0 0 0 0 0 </pose>
             <visualize>true</visualize>
@@ -66,13 +65,25 @@
                 <frame_name>camera_optical_link</frame_name>
             </plugin>
+        </sensor> -->
+        <sensor name="camera" type="camera">
+            <pose> 0 0 0 0 0 0 </pose>
+            <visualize>true</visualize>
+            <update_rate>10</update_rate>
+            <camera>
+                <camera_info_topic>camera/camera_info</camera_info_topic>
+                <horizontal_fov>1.089</horizontal_fov>
+                <image>
+                    <format>R8G8B8</format>
+                    <width>640</width>
+                    <height>480</height>
+                </image>
+                <clip>
+                    <near>0.05</near>
+                    <far>8.0</far>
+                </clip>
+            </camera>
+            <topic>camera/image_raw</topic>
+            <gz_frame_id>camera_link_optical</gz_frame_id>
         </sensor>
     </gazebo>
-    <gazebo reference="camera_link">
-        <visual>
-            <geometry>
-                <mesh filename="package://rom_ur_sim/meshes/sensors/camera/kinetic.stl"/>
-            </geometry>
-            <material>Gazebo/Red</material>
-        </visual>
-    </gazebo>
 </robot>

File: ur5/rom_ur_sim/urdf/ur5_camera_gripper.urdf.xacro (robot description, xacro)
@@ -4,5 +4,5 @@
    <xacro:arg name="name" default="ur"/>
    <!-- import main macro -->
-   <xacro:include filename="$(find rom_ur_sim)/urdf/camera.xacro"/>
+   <xacro:include filename="$(find rom_ur_sim)/urdf/camera_ign.xacro"/>
    <xacro:include filename="$(find rom_ur_sim)/urdf/ur5_macro.xacro"/>
    <!-- possible 'ur_type' values: ur3, ur3e, ur5, ur5e, ur7e, ur10, ur10e, ur12e, ur16e, ur15, ur20, ur30 -->

Commit message: to convert cpp

File: ur5/rom_ur_sim/urdf/camera_ign.xacro (robot description, xacro)
@@ -17,5 +17,5 @@
                 <mesh filename="package://rom_ur_sim/meshes/sensors/camera/kinetic.stl"/>
             </geometry>
-            <material name="red"/>
+            <material name="Blue"/>
         </visual>
         <collision>
@@ -29,5 +29,5 @@
         <parent link="base_link"/>
         <child link="camera_link"/>
-        <origin xyz="0.5 0 1.2" rpy="0 1.57 0" />
+        <origin xyz="0.5 0 0.7" rpy="0 1.57 0" />
     </joint>
     <link name="camera_optical_link"></link>

Commit message: ready to grasping object

File: ur5/rom_ur_sim/urdf/camera_ign.xacro (robot description, xacro)
@@ -29,5 +29,6 @@
         <parent link="base_link"/>
         <child link="camera_link"/>
-        <origin xyz="0.2 0.6 1.2" rpy="0 1.570796326 0" />
+        <!-- <origin xyz="0.2 0.6 1.2" rpy="0 1.570796326 0" /> -->
+        <origin xyz="0 0 1.2" rpy="0 1.57 0" />
     </joint>
     <link name="camera_optical_link"></link>
@@ -36,4 +37,5 @@
         <child link="camera_optical_link"/>
         <origin xyz="0 0 0" rpy="-1.57 0 -1.57" />
+        <!-- <origin xyz="0 0 0" rpy="0 0 0" /> -->
     </joint>
     <gazebo reference="camera_link">
