Commit message: moveit done, not get motion planning

File: ur5/rom_ur5_moveit_config/config/ur.ros2_control.xacro (robot description, xacro)
@@ -2,5 +2,5 @@
 <robot xmlns:xacro="http://www.ros.org/wiki/xacro">
     <xacro:macro name="ur_ros2_control" params="name initial_positions_file">
-        <xacro:property name="initial_positions" value="${load_yaml(initial_positions_file)['initial_positions']}"/>
+        <xacro:property name="initial_positions" value="${xacro.load_yaml(initial_positions_file)['initial_positions']}"/>
         <ros2_control name="${name}" type="system">
             <hardware>

File: ur5/rom_ur5_moveit_config/config/ur.urdf.xacro (robot description, xacro)
@@ -5,5 +5,5 @@
     <xacro:include filename="$(find rom_ur_sim)/urdf/ur5_camera_gripper.urdf.xacro" />
     <!-- Import control_xacro -->
-    <!-- <xacro:include filename="ur.ros2_control.xacro" />
-    <xacro:ur_ros2_control name="FakeSystem" initial_positions_file="$(arg initial_positions_file)"/> -->
+    <!-- <xacro:include filename="ur.ros2_control.xacro" /> -->
+    <!-- <xacro:ur_ros2_control name="FakeSystem" initial_positions_file="$(arg initial_positions_file)"/> -->
 </robot>

File: ur5/rom_ur_sim/urdf/ur5_camera.urdf.xacro (robot description, xacro)
@@ -4,5 +4,5 @@
    <xacro:arg name="name" default="ur"/>
    <!-- import main macro -->
-   <xacro:include filename="$(find rom_ur_sim)/urdf/camera_ign.xacro"/>
+   <!-- <xacro:include filename="$(find rom_ur_sim)/urdf/camera_ign.xacro"/> -->
    <xacro:include filename="$(find rom_ur_sim)/urdf/ur5_macro.xacro"/>
    <xacro:include filename="$(find ur_simulation_gz)/urdf/ur_gz.ros2_control.xacro" />
